Commit message: Add files via upload

File: description/robot_core.xacro (robot description, xacro)
@@ -34,4 +34,12 @@
         </xacro:inertial_box>
     </link>
+    <!-- base footprint -->
+    <joint name="base_footprint_joint" type="fixed">
+        <parent link="base_link"/>
+        <child link="base_footprint"/>
+        <origin xyz="0 0 0" rpy="0 0 0"/>
+    </joint>
+    <link name="base_footprint">
+    </link>
     <!-- chassis -->
     <!-- <joint name="chassis_joint" type="fixed">
