Commit message: Add files via upload

File: description/lidar.xacro (robot description, xacro)
@@ -1,6 +1,9 @@
 <?xml version="1.0"?>
 <robot xmlns:xacro="http://www.ros.org/wiki/xacro">
+    <material name="red">
+        <color rgba="1 0 0 1"/>
+    </material>
     <joint name="laser_joint" type="fixed">
-        <parent link="base_link"/>
+        <parent link="chassis"/>
         <child link="laser_frame"/>
         <origin xyz="0 0 0.14" rpy="0 0 0"/>

File: description/robot_core.xacro (robot description, xacro)
@@ -16,4 +16,20 @@
     <!-- base link -->
     <link name="base_link">
+    </link>
+    <!-- base footprint -->
+    <joint name="base_footprint_joint" type="fixed">
+        <parent link="base_link"/>
+        <child link="base_footprint"/>
+        <origin xyz="0 0 0" rpy="0 0 0"/>
+    </joint>
+    <link name="base_footprint">
+    </link>
+    <!-- chassis -->
+    <joint name="chassis_joint" type="fixed">
+        <parent link="base_link"/>
+        <child link="chassis"/>
+        <origin xyz="0 0 0" rpy="0 0 0"/>
+    </joint>
+    <link name="chassis">
         <visual>
         <origin xyz="0 0 0.095"/>
@@ -34,20 +50,4 @@
         </xacro:inertial_box>
     </link>
-    <!-- base footprint -->
-    <joint name="base_footprint_joint" type="fixed">
-        <parent link="base_link"/>
-        <child link="base_footprint"/>
-        <origin xyz="0 0 0" rpy="0 0 0"/>
-    </joint>
-    <link name="base_footprint">
-    </link>
-    <!-- chassis -->
-    <!-- <joint name="chassis_joint" type="fixed">
-        <parent link="base_link"/>
-        <child link="chassis"/>
-        <origin xyz="0.0 0.0 0.0"/>
-    </joint>
-    <link name="chassis">
-    </link> -->
     <!-- left wheel -->
     <joint name="left_wheel_joint" type="continuous">
@@ -167,5 +167,5 @@
     <!-- front caster wheel -->
     <joint name="front_caster_joint" type="fixed">
-        <parent link="base_link"/>
+        <parent link="chassis"/>
         <child link="front_caster_wheel"/>
         <origin xyz="0.06 0 0.005"/>
@@ -256,5 +256,5 @@
     <!-- rear caster wheel -->
     <joint name="rear_caster_joint" type="fixed">
-        <parent link="base_link"/>
+        <parent link="chassis"/>
         <child link="rear_caster_wheel"/>
         <origin xyz="-0.06 0 0.005"/>
